File: pcb/microsd/microsd.kicad_pcb (KiCad board)
At the start: 2 copper layers, 0 parts

Commit message: [microsd] add v1 microsd
Parts:
- added C1: 22uf/25V, Capacitor_SMD:C_0805_2012Metric, F.Cu at (60.3, 60.4)
- added C2: 0.1uf/50v, Capacitor_SMD:C_0603_1608Metric, F.Cu at (62.3, 60.4)
- added J1: Micro_SD_Card_Det_Hirose_DM3AT, !Misc:HRS_DM3AT-SF-PEJM5, F.Cu at (72.5, 58.8)
- added PM1: PMOD_Dual_Male, !Misc:PMOD_Dual_Male, F.Cu at (49.2, 52.4)
- added R1: 20K, Resistor_SMD:R_0603_1608Metric, F.Cu at (56.4, 52.1)
- added R2: 20K, Resistor_SMD:R_0603_1608Metric, F.Cu at (56.4, 54.0)
- added R3: 20K, Resistor_SMD:R_0603_1608Metric, F.Cu at (56.4, 55.9)
- added R4: 20K, Resistor_SMD:R_0603_1608Metric, F.Cu at (56.4, 59.7)
- added R5: 20K, Resistor_SMD:R_0603_1608Metric, F.Cu at (56.4, 57.8)
- added R6: 20K, Resistor_SMD:R_0603_1608Metric, F.Cu at (56.4, 61.6)
- added R7: 20K, Resistor_SMD:R_0603_1608Metric, F.Cu at (56.4, 63.5)
- added R8: 240, Resistor_SMD:R_0603_1608Metric, F.Cu at (56.4, 65.4)
Routing:
- net /DAT1: track 0.00 -> 25.3 mm, vias 0 -> 2
- net /CS/CD/DAT3: track 0.00 -> 24.2 mm, vias 0 -> 2
- net /DAT2: track 0.00 -> 24.1 mm, vias 0 -> 2
- net /MISO/DAT0/DO: track 0.00 -> 22.6 mm, vias 0 -> 2
- net /MOSI/CMD/DI: track 0.00 -> 21.2 mm, vias 0 -> 2
- net /CD: track 0.00 -> 20.2 mm
- net +3V3: track 0.00 -> 18.0 mm, vias 0 -> 9
- net /SCLK/CLK: track 0.00 -> 17.0 mm, vias 0 -> 2
- net GND: track 0.00 -> 10.6 mm, vias 0 -> 7
- net Net-(J1-DET_A): track 0.00 -> 7.65 mm
- added copper zone on In2.Cu, net +3V3
- added copper zone on In1.Cu, net GND
Other:
- board outline added: 38.1 x 20.3 mm
- copper layers 2 -> 4
- board text added: "https://github.com/pbozeman/pmods"
- board text added: "v1"
