File: pcb/microsd/microsd.kicad_sch (KiCad schematic)
At the start: 0 parts

Commit message: [microsd] add v1 microsd
Parts:
- added C1: 22uf/25V, Capacitor_SMD:C_0805_2012Metric, symbol !Misc:C_22uf_0805
- added C2: 0.1uf/50v, Capacitor_SMD:C_0603_1608Metric, symbol !Misc:C_0.1uf_0603
- added J1: Micro_SD_Card_Det_Hirose_DM3AT, !Misc:HRS_DM3AT-SF-PEJM5, symbol !Misc:Micro_SD_Card_Det_Hirose_DM3AT
- added PM1: PMOD_Dual_Male, !Misc:PMOD_Dual_Male, symbol !Misc:PMOD_Dual_Male
- added R1, R2, R3, R4, R5, R6, R7: 20K, Resistor_SMD:R_0603_1608Metric, symbol !Misc:R_20K_0603
- added R8: 240, Resistor_SMD:R_0603_1608Metric, symbol !Misc:R_240_0603
Connections:
- new net: J1.10 (DET_A), R8.2
- new net +3V3: C1.1, C2.1, J1.4 (VDD), PM1.12 (VCC), PM1.6 (VCC), R1.1, R2.1, R3.1, R4.1, R5.1, R6.1, R7.1
- new net CD: PM1.9, R7.2, R8.1
- new net CS/CD/DAT3: J1.2 (DAT3/CD), PM1.1, R1.2
- new net DAT1: J1.8 (DAT1), PM1.7, R6.2
- new net DAT2: J1.1 (DAT2), PM1.8, R2.2
- new net GND: C1.2, C2.2, J1.11 (SHIELD), J1.6 (VSS), J1.9 (DET_B), PM1.11 (GND), PM1.5 (GND)
- new net MISO/DAT0/DO: J1.7 (DAT0), PM1.3, R5.2
- new net MOSI/CMD/DI: J1.3 (CMD), PM1.2, R3.2
- new net NC/EN: PM1.10
- new net SCLK/CLK: J1.5 (CLK), PM1.4, R4.2
